Commit message: fix(nav2): align URDF root + AMCL base_frame_id to base_link (matches Carter sim)
Carter's Nova_Carter_ROS USD publishes /tf with child_frame_id=base_link
(odom -> base_link). The URDF had base_footprint as the root, which
introduced a parallel TF chain that didn't connect to the sim's. Nav2
AMCL with base_frame_id: base_footprint couldn't find any TF chain
to base_footprint, so it never published map -> odom and Nav2 rejected
goals with 'map frame does not exist'.

Fix: drop base_footprint, make base_link the URDF root, point AMCL's
base_frame_id at base_link. Now the chain is:
  map (AMCL) -> odom (sim) -> base_link (sim) -> laser_frame (RSP)

Found via M1 smoke debug — see [[feedback-foundationpose-install-gotchas]]
... actually a Nav2 gotcha, not FP. Worth adding to the project memory.

Co-Authored-By: Claude Opus 4.7 (1M context) <noreply@anthropic.com>

File: ros2_ws/src/wdt_carter_description/urdf/carter.urdf.xacro (robot description, xacro)
@@ -2,17 +2,20 @@
 <!--
   Nova Carter URDF for Nav2 footprint + TF chain.
-  Isaac Sim ships Nova Carter with its own physics + sensors. This URDF
-  exists only so ROS2-side consumers (Nav2's costmaps, RViz, MoveIt2
-  scene monitor) have a consistent footprint and frame tree:
-    base_footprint  →  base_link  →  laser_frame
-  All three frames are also published by the sim-side OmniGraph (Task 6)
-  so robot_state_publisher and the sim agree on TF.
+  Isaac Sim's Nova Carter USD publishes /tf with `odom → base_link`,
+  so this URDF makes `base_link` the root and chains the static
+  per-sensor frames off it:
+    odom (from sim) → base_link → laser_frame
   The chassis collision/visual is approximated as a 0.6 × 0.4 × 0.5 m
   box. The actual Carter geometry is more complex; Nav2's costmap only
   needs an inflation-radius-friendly footprint, so the box is sufficient.
+  Note: Phase 1 had a `base_footprint` root with `base_footprint →
+  base_link` fixed joint, intended to follow the typical Nav2 mobile
+  convention. But Isaac Sim publishes the dynamic transform with
+  `child_frame_id: base_link`, not `base_footprint`, breaking the TF
+  chain (M1 smoke debug 2026-05-15). Drop base_footprint and use
+  base_link as both the URDF root and AMCL's `base_frame_id`.
 -->
 <robot xmlns:xacro="http://www.ros.org/wiki/xacro" name="nova_carter">
   <xacro:arg name="robot_namespace" default=""/>
-  <link name="base_footprint"/>
   <link name="base_link">
     <visual>
@@ -25,9 +28,4 @@
     </collision>
   </link>
-  <joint name="base_footprint_to_base_link" type="fixed">
-    <parent link="base_footprint"/>
-    <child link="base_link"/>
-    <origin xyz="0 0 0"/>
-  </joint>
   <link name="laser_frame"/>
   <joint name="base_link_to_laser" type="fixed">
